File: SwitchBox.kicad_pcb (KiCad board)
At the start: 2 copper layers, 150 x 191 mm, 93 parts, among them Q1 BS250, Q2 BS250, Q3 BS250, Q4 BS250, Q5 BS250, Q6 BS250, Q7 BS250, Q8 BS250

Commit message: Edits
Parts:
- added G***: LOGO, additions:QRcode_Smaller, B.Cu at (80.6, 146.7)
- moved BLACK 7.65 mm to (68.5, 216.6)
- moved RED 7.65 mm to (68.5, 37.6)
- moved BLACK 5.59 mm to (43.3, 216.6)
- moved BLACK 5.29 mm to (144.1, 216.2)
- moved RED 5.29 mm to (144.1, 37.6)
- moved BLACK 5.21 mm to (169.3, 216.2)
- moved RED 5.14 mm to (43.3, 37.6)
- moved RED 5.13 mm to (169.3, 37.6)
- moved BLACK 3.34 mm to (93.7, 216.2)
- moved RED 3.34 mm to (93.7, 37.6)
- moved BLACK 1.00 mm to (176.2, 50.2)
- moved BLACK 1.00 mm to (176.2, 79.1)
- moved BLACK 1.00 mm to (176.2, 91.4)
- moved BLACK 1.00 mm to (176.2, 120.4)
- moved BLACK 1.00 mm to (176.2, 132.7)
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Routing:
- net Net-(J1-Pad1): track 158.3 -> 150.2 mm
- net Net-(J10-Pad1): track 157.9 -> 154.0 mm
